File: pcb/PowerSupply.kicad_sch (KiCad schematic)
At the start: 71 parts, among them Q1 Q_NMOS_GDS, Q2 Q_NMOS_GDS, Q3 Q_NMOS_GDS, Q4 Q_NMOS_GDS, Q5 Q_NMOS, Q6 Q_NMOS, Q7 Q_NMOS, Q8 Q_NMOS, U1 LM5176PWP, U2 RK097111080R

Commit message: 频率，指示灯电路
Parts:
- added C32: 100n, symbol Device:C
- added C33: 1n, symbol Device:C
- added D6: SS310, Diode_SMD:D_SMA, symbol Diode:SS310
- added D7: LED, symbol Device:LED
- added R25: 1.5k, symbol Device:R
- added R26: 5.1k, symbol Device:R
- added RV1, RV2: 100k, symbol Device:R_Potentiometer
Connections:
- net powerPAD is gone; now on net GND: U1.29 (PowerPAD)
- net BOOT2: now also C32.2, D6.1 (K)
- net GND: now also C33.1, D7.1 (K), R25.1, RV2.3
- net LM5176_VOUT: now also R26.2, RV1.1, RV1.2
- net SW1: now also L2.1, Q5.S, Q8.D
- net VCC: now also D6.2 (A)
- net fb: no longer U1.11 (FB)
- net pgood: no longer U1.17 (PGOOD)
- net q4-2: no longer U1.18 (SW2)
- net rt/sync: no longer U1.6 (RT/SYNC)
- net SW2: now reaches L2.2, Q6.S, Q7.D
- net SW2: now also U1.18 (SW2), C32.1
- new net FB: R25.2, RV1.3, U1.11 (FB)
- new net PGOOD: D7.2 (A), R26.1, U1.17 (PGOOD)
- new net RT_SYNC: C33.2, RV2.1, RV2.2, U1.6 (RT/SYNC)
Other:
- note added: "PGOOD指示灯"
- note added: "开关频率调节 这里的电位器已经超出范围， 暂时不管"
- note added: "电压反馈"
- note added: "自举电容， 驱动H部分MOS 二极管需耐压55V 电容耐压16V"
- note added: "还没画完>"
- note removed: "自举电容， 驱动H部分MOS 二极管需耐压55V"
