File: pcb/PowerSupply.kicad_sch (KiCad schematic)
At the start: 79 parts, among them Q1 Q_NMOS_GDS, Q2 Q_NMOS_GDS, Q3 Q_NMOS_GDS, Q4 Q_NMOS_GDS, Q5 Q_NMOS, Q6 Q_NMOS, Q7 Q_NMOS, Q8 Q_NMOS, U1 LM5176PWP, U2 RK097111080R

Commit message: 限流，抖动
Parts:
- added C34: 10n, symbol Device:C
- added C35: 1u, symbol Device:C
- added R27, R28: 100, symbol Device:R
- added R29: 8m, symbol Device:R
- R23, R24: value 10R -> 100
Connections:
- net GND: now also C34.1; no longer U1.5 (DITH)
- net LM5176_VOUT: now also R27.1, R29.2
- net isns+: no longer U1.14 (ISNS(+))
- net isns-: no longer U1.13 (ISNS(-))
- net at Q6.D: now also R28.1, R29.1
- new net DITH: C34.2, U1.5 (DITH)
- new net ISNS+: C35.1, R28.2, U1.14 (ISNS(+))
- new net ISNS-: C35.2, R27.2, U1.13 (ISNS(-))
Other:
- note added: "输入电压检测脚 2k电阻只在vo大于40V时需要"
- note added: "输出电流感知 （限流电路） 采样电阻暂时短接"
- note added: "频率抖动"
- note removed: "输入电压检测脚"
- moved on the sheet: C31, L2, Q5, Q6, Q7, Q8, R22, R23, R24

Commit message: 很多东西
Parts:
- removed C33: 1n, symbol Device:C
- added C36, C37, C38, C39, C40: 4.7u, symbol Device:C
- added C41, C42, C43, C44: 22u, symbol Device:C
- added C45, C46, C47, C48, C49: 1u, symbol Device:C
- added C50, C51, C52: 100u, symbol Device:C
Connections:
- net GNDPWR: now also C36.1, C37.1, C38.1, C39.1, C40.1, C41.1, C42.1, C43.1, C44.1, C45.1, C46.1, C47.1, C48.1, C49.1, C50.1, C51.1, C52.1
- net LM5176_VOUT: now also C45.2, C46.2, C47.2, C48.2, C49.2, C50.2, C51.2, C52.2
- net USB_VBUS: now also C36.2, C37.2, C38.2, C39.2, C40.2, C41.2, C42.2, C43.2, C44.2
Other:
- note added: "PGOOD上拉+ PGOOD指示灯"
- note added: "电压反馈（调电压）"
- note added: "输入滤波 电容最低20V"
- note added: "输出滤波 电容最低55V"
- note removed: "PGOOD指示灯"
- note removed: "电压反馈"
- note removed: "还没画完>"
- moved on the sheet: C35, D7, R26, R27, R28, R29

Commit message: 很多东西
Parts:
- removed C1: 560p, symbol Device:C
- removed C10, C11, C12, C13, C14: 10u, symbol Device:C
- removed C15, C16: 180u, symbol Device:C
- removed C17, C18, C19, C20, C21, C22: 4.7u, symbol Device:C
- removed C2: 33n, symbol Device:C
- removed C23, C24, C4, C5, C8: 0.1u, symbol Device:C
- removed C25: 220p, symbol Device:C
- removed C3, C9: 1u, symbol Device:C
- removed C6: 1n, symbol Device:C
- removed C7: 68u, symbol Device:C
- removed D1: D, symbol Device:D
- removed D2, D3: (no value), Diode_THT:D_DO-41_SOD81_P10.16mm_Horizontal, symbol Diode:1N47xxA
- removed L1: 4.7u, symbol Device:L
- removed Q1: Q_NMOS_GDS, Package_DFN_QFN:DFN-8-1EP_6x5mm_P1.27mm_EP2x2mm, symbol Transistor_FET:Q_NMOS_GDS
- removed Q2, Q3, Q4: Q_NMOS_GDS, symbol Transistor_FET:Q_NMOS_GDS
- removed R1, R4, R8: 10k, symbol Device:R
- removed R10, R11, R13, R14: 100, symbol Device:R
- removed R12: 8m, symbol Device:R
- removed R15: 1.5k, symbol Device:R
- removed R2: 27.4k, symbol Device:R
- removed R3: 93.1k, symbol Device:R
- removed R5: 59.0k, symbol Device:R
- removed R6: 249k, symbol Device:R
- removed R7: 2k, symbol Device:R
- removed R9: 0, symbol Device:R
- removed U2: RK097111080R, easyeda2kicad:RES-ADJ-TH_RK097111080R, symbol easyeda2kicad:RK097111080R
- added C53: 240p, symbol Device:C
- added C54: 33n, symbol Device:C
- added C55: 560p, symbol Device:C
- added R30: 10k, symbol Device:R
Connections:
- net GND: now also C53.1, C55.1, R30.1
- net comp renamed COMP
- net COMP: now also C54.2, C55.2
- net slope renamed SLOPE
- net SLOPE: now also C53.2
- new net: C54.1, R30.2
Other:
- note added: "VCC滤波 VCC用于充电两个自举电容"
- note added: "斜坡补偿 用于抑制D超过50%时的震荡"
- note added: "频率补偿"
- note removed: "VCC滤波"
- moved on the sheet: C26, C27, C28, C29, C30, C31, C32, C34, C35, C36, C37, C38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

Commit message: 所有封装
Parts:
- removed C41, C42, C43, C44: 22u, symbol Device:C
- removed C50, C51, C52: 100u, symbol Device:C
- added C1, C3, C4: 22u 20V, Capacitor_SMD:CP_Elec_5x5.4, symbol Device:C_Polarized
- added C2: 22u 20V, Capacitor_SMD:C_Elec_5x5.4, symbol Device:C_Polarized
- added C5, C6, C7: 100u 50V, Capacitor_SMD:CP_Elec_10x10.5, symbol Device:C_Polarized
- C26, C27, C28, C29, C30, C31, C32, C34, C35, C36, C37, C38, C39, C40, C53, C54, C55: footprint (none) -> Capacitor_SMD:C_0805_2012Metric
- C45, C46, C47, C48, C49: footprint (none) -> Capacitor_SMD:C_1206_3216Metric
- D7: footprint (none) -> LED_SMD:LED_0805_2012Metric
- L2: footprint (none) -> Inductor_SMD:L_TaiTech_TMPC1265_13.5x12.5mm
- Q5, Q6, Q7, Q8: footprint (none) -> lcsc_pro:TDSON-8_L5.9-W5.2-P1.27-BL-1
- R16, R17, R18, R19, R21, R23, R24, R25, R26, R27, R28, R30: footprint (none) -> Resistor_SMD:R_1206_3216Metric
- R22, R29: footprint (none) -> Resistor_SMD:R_2512_6332Metric
- RV1, RV2: footprint (none) -> lcsc_pro:RES-ADJ-TH_RK097111080R
Connections:
- net GNDPWR: now also C1.2, C2.2, C3.2, C4.2, C6.2, C7.2
- net LM5176_VOUT: now also C6.1, C7.1
- net USB_VBUS: now also C1.1, C2.1, C3.1, C4.1

Commit message: 调整元件参数
Parts:
- removed C1, C3, C4: 22u 20V, Capacitor_SMD:CP_Elec_5x5.4, symbol Device:C_Polarized
- removed C2: 22u 20V, Capacitor_SMD:C_Elec_5x5.4, symbol Device:C_Polarized
- removed C36, C37, C38, C39, C40: 4.7u, Capacitor_SMD:C_0805_2012Metric, symbol Device:C
- removed C46, C47, C48, C49: 1u, Capacitor_SMD:C_1206_3216Metric, symbol Device:C
- removed C6, C7: 100u 50V, Capacitor_SMD:CP_Elec_10x10.5, symbol Device:C_Polarized
- added C10, C11, C15, C16, C18, C19, C20, C21, C9: 2.2u 100V, Capacitor_SMD:C_1206_3216Metric, symbol Device:C
- added C24, C25, C26, C27, C28, C29: 100u 63V, Capacitor_SMD:CP_Elec_8x10.5, symbol Device:C_Polarized
- C17: renamed from C55; value 560p -> 330p
- C22: renamed from C53; value 240p -> 470p
- C23: renamed from C5; value 100u 50V -> 100u 63V; footprint Capacitor_SMD:CP_Elec_10x10.5 -> Capacitor_SMD:CP_Elec_8x10.5
- C4: renamed from C26; value 100n -> 330n
- C8: renamed from C45; value 1u -> 2.2u 100V
- R12: renamed from R30; value 10k -> 20k
- R3: renamed from R16; value 470k -> 249k
- R4: renamed from R17; value 130k -> 75k
- renumbered C31 to C1, C54 to C12, C30 to C13, C34 to C14, C28 to C2, C27 to C3, C29 to C5, C32 to C6, C35 to C7, D4 to D1, D5 to D2, D6 to D3, D7 to D4, L2 to L1, Q5 to Q1, Q8 to Q2, Q6 to Q3, Q7 to Q4, R23 to R1, R19 to R10, R27 to R11, R25 to R13, R26 to R14, R24 to R2, R18 to R5, R22 to R6, R21 to R7, R28 to R8, R29 to R9, RV2 to RV1, RV1 to RV2
Connections:
- net GNDPWR: now also C23.2, C10.1, C11.1, C15.1, C16.1, C18.1, C19.1, C20.1, C21.1, C24.2, C25.2, C26.2, C27.2, C28.2, C29.2, C9.1
- net LM5176_VOUT: now also C23.1, C10.2, C15.2, C18.2, C20.2, C25.1, C26.1, C27.1, C28.1, C29.1
- net USB_VBUS: now also C11.2, C16.2, C19.2, C21.2, C24.1, C9.2
Other:
- moved on the sheet: C23

Commit message: 翻译指南
Parts:
- R6, R9: value 8m -> 3m
Changed lines of the file:
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@@
 			)
 		)
-		(property "Value" "8m"
+		(property "Value" "3m"
 			(at 48.26 180.34 0)
 			(show_name no)
@@
 			)
 		)
-		(property "Value" "8m"
+		(property "Value" "3m"
 			(at 93.218 134.874 90)
 			(show_name no)

Commit message: 总开关电路
Parts:
- added D6: D_Zener, Diode_SMD:D_SOD-123, symbol Device:D_Zener
- added Q5: PMOS, lcsc_pro:DFN-8_L5.8-W4.9-P1.27-LS6.1-BL-2, symbol Simulation_SPICE:PMOS
- added R24, R25: 5.1k, Resistor_SMD:R_1206_3216Metric, symbol Device:R
- added SW1: SW_Push_DPDT, lcsc_pro:SW-SMD_6P-L9.1-W3.5-P2.50, symbol Switch:SW_Push_DPDT
- L1: value 4.7u -> 3.3u
Connections:
- net GND: now also R25.1
- net USB_VBUS: now also D6.1 (K), Q5.3 (S), R24.2; no longer C11.2, C16.2, C19.2, C21.2, C24.1, C9.2, D1.2 (A), Q1.D, R10.2, R3.2
- new net: R24.1, SW1.1 (A), SW1.4 (A)
- new net: D6.2 (A), Q5.2 (G), SW1.2 (B), SW1.5 (B)
- new net: R25.2, SW1.3 (C), SW1.6 (C)
- new net INPUT: C11.2, C16.2, C19.2, C21.2, C24.1, C9.2, D1.2 (A), Q1.D, Q5.1 (D), R10.2, R3.2
Other:
- note added: "使用PMOS的开关，稳压管用来防止GS击穿"
