File: pcb/PowerSupply.kicad_sch (KiCad schematic)
At the start: 60 parts, among them Q1 Q_NMOS, Q2 Q_NMOS, Q3 Q_NMOS, Q4 Q_NMOS, Q5 PMOS, SW1 SW_Push_DPDT, U1 LM5176PWP

Commit message: 整理封装
Parts:
- removed Q5: PMOS, lcsc_pro:DFN-8_L5.8-W4.9-P1.27-LS6.1-BL-2, symbol Simulation_SPICE:PMOS
- added Q6: Q_PMOS, custom_lib:DFN-8_L5.8-W4.9-P1.27-LS6.1-BL-2, symbol Device:Q_PMOS
- Q1, Q2, Q3, Q4: footprint lcsc_pro:TDSON-8_L5.9-W5.2-P1.27-BL-1 -> custom_lib:TDSON-8_L5.9-W5.2-P1.27-BL-1
- RV1, RV2: footprint lcsc_pro:RES-ADJ-TH_RK097111080R -> custom_lib:RES-ADJ-TH_RK097111080R
- SW1: footprint lcsc_pro:SW-SMD_6P-L9.1-W3.5-P2.50 -> custom_lib:SW-SMD_6P-L9.1-W3.5-P2.50
Connections:
- net INPUT: now also Q6.D
- net USB_VBUS: now also Q6.S
- net at D6.2 (A), SW1.2 (B), SW1.5 (B): now also Q6.G
Changed lines of the file:
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@@
 			)
 		)
-		(property "Footprint" "lcsc_pro:RES-ADJ-TH_RK097111080R"
+		(property "Footprint" "custom_lib:RES-ADJ-TH_RK097111080R"
 			(at 201.93 128.27 0)
 			(hide yes)
@@
 			)
 		)
-		(property "Footprint" "lcsc_pro:TDSON-8_L5.9-W5.2-P1.27-BL-1"
+		(property "Footprint" "custom_lib:TDSON-8_L5.9-W5.2-P1.27-BL-1"
 			(at 62.23 157.48 0)
 			(hide yes)
@@
 			)
 		)
-		(property "Footprint" "lcsc_pro:TDSON-8_L5.9-W5.2-P1.27-BL-1"
+		(property "Footprint" "custom_lib:TDSON-8_L5.9-W5.2-P1.27-BL-1"
 			(at 62.23 139.7 0)
 			(hide yes)
@@
 			)
 		)
-		(property "Footprint" "lcsc_pro:SW-SMD_6P-L9.1-W3.5-P2.50"
+		(property "Footprint" "custom_lib:SW-SMD_6P-L9.1-W3.5-P2.50"
 			(at 189.23 233.68 0)
 			(hide yes)
@@
 			)
 		)
-		(property "Footprint" "lcsc_pro:TDSON-8_L5.9-W5.2-P1.27-BL-1"
+		(property "Footprint" "custom_lib:TDSON-8_L5.9-W5.2-P1.27-BL-1"
 			(at 41.91 139.7 0)
 			(hide yes)
@@
 	)
 	(symbol
+		(lib_id "Device:Q_PMOS")
+		(at 158.75 243.84 180)
+		(unit 1)
+		(body_style 1)
+		(exclude_from_sim no)
+		(in_bom yes)
+		(on_board yes)
+		(in_pos_files yes)
+		(dnp no)
+		(fields_autoplaced yes)
+		(property "Reference" "Q6"
+			(at 152.4 242.5699 0)
+			(show_name no)
+			(do_not_autoplace no)
+			(effects
+				(font
+					(size 1.27 1.27)
+				)
+				(justify left)
+			)
+		)
+		(property "Value" "Q_PMOS"
+			(at 152.4 245.1099 0)
+			(show_name no)
+			(do_not_autoplace no)
+			(effects
+				(font
+					(size 1.27 1.27)
+				)
+				(justify left)
+			)
+		)
+		(property "Footprint" "custom_lib:DFN-8_L5.8-W4.9-P1.27-LS6.1-BL-2"
+			(at 153.67 246.38 0)
+			(hide yes)
+			(show_name no)
+			(do_not_autoplace no)
+			(effects
+				(font
+					(size 1.27 1.27)
+				)
+			)
+		)
+		(property "Datasheet" ""
+			(at 158.75 243.84 0)
+			(hide yes)
+			(show_name no)
+			(do_not_autoplace no)
+			(effects
+				(font
+					(size 1.27 1.27)
+				)
+			)
+		)
+		(property "Description" "P-MOSFET transistor"
+			(at 158.75 243.84 0)
+			(hide yes)
+			(show_name no)
+			(do_not_autoplace no)
+			(effects
+				(font
+					(size 1.27 1.27)
+				)
+			)
+		)
+		(pin "D"
+		)
+		(pin "S"
+		)
+		(pin "G"
+		)
+		(instances
+			(project "PowerSupply"
+				(path "/3ecbe32c-4290-401a-9b8c-a7a0b4ba8879"
+					(reference "Q6")
+					(unit 1)
+				)
+			)
+		)
+	)
+	(symbol
 		(lib_id "Device:R")
 		(at 201.93 139.7 180)
@@
 	)
 	(symbol
-		(lib_id "Simulation_SPICE:PMOS")
-		(at 158.75 243.84 180)
-		(unit 1)
-		(body_style 1)
-		(exclude_from_sim no)
-		(in_bom yes)
-		(on_board yes)
-		(in_pos_files yes)
-		(dnp no)
-		(fields_autoplaced yes)
-		(property "Reference" "Q5"
-			(at 152.4 242.5699 0)
-			(show_name no)
-			(do_not_autoplace no)
-			(effects
-				(font
-					(size 1.27 1.27)
-				)
-				(justify left)
-			)
-		)
-		(property "Value" "PMOS"
-			(at 152.4 245.1099 0)
-			(show_name no)
-			(do_not_autoplace no)
-			(effects
-				(font
-					(size 1.27 1.27)
-				)
-				(justify left)
-			)
-		)
-		(property "Footprint" "lcsc_pro:DFN-8_L5.8-W4.9-P1.27-LS6.1-BL-2"
-			(at 153.67 246.38 0)
-			(hide yes)
-			(show_name no)
-			(do_not_autoplace no)
-			(effects
-				(font
-					(size 1.27 1.27)
-				)
-			)
-		)
-		(property "Datasheet" "https://ngspice.sourceforge.io/docs/ngspice-html-manual/manual.xhtml#cha_MOSFETs"
-			(at 158.75 231.14 0)
-			(hide yes)
-			(show_name no)
-			(do_not_autoplace no)
-			(effects
-				(font
-					(size 1.27 1.27)
-				)
-			)
-		)
-		(property "Description" "P-MOSFET transistor, drain/source/gate"
-			(at 158.75 243.84 0)
-			(hide yes)
-			(show_name no)
-			(do_not_autoplace no)
-			(effects
-				(font
-					(size 1.27 1.27)
-				)
-			)
-		)
-		(property "Sim.Device" "PMOS"
-			(at 158.75 226.695 0)
-			(hide yes)
-			(show_name no)
-			(do_not_autoplace no)
-			(effects
-				(font
-					(size 1.27 1.27)
-				)
-			)
-		)
-		(property "Sim.Type" "VDMOS"
-			(at 158.75 224.79 0)
-			(hide yes)
-			(show_name no)
-			(do_not_autoplace no)
-			(effects
-				(font
-					(size 1.27 1.27)
-				)
-			)
-		)
-		(property "Sim.Pins" "1=D 2=G 3=S"
-			(at 158.75 228.6 0)
-			(hide yes)
-			(show_name no)
-			(do_not_autoplace no)
-			(effects
-				(font
-					(size 1.27 1.27)
-				)
-			)
-		)
-		(pin "1"
-		)
-		(pin "2"
-		)
-		(pin "3"
-		)
-		(instances
-			(project "PowerSupply"
-				(path "/3ecbe32c-4290-401a-9b8c-a7a0b4ba8879"
-					(reference "Q5")
-					(unit 1)
-				)
-			)
-		)
-	)
-	(symbol
 		(lib_id "Device:C")
 		(at 204.47 93.98 180)
@@
 			)
 		)
-		(property "Footprint" "lcsc_pro:RES-ADJ-TH_RK097111080R"
+		(property "Footprint" "custom_lib:RES-ADJ-TH_RK097111080R"
 			(at 34.29 217.17 0)
 			(hide yes)
@@
 			)
 		)
-		(property "Footprint" "lcsc_pro:TDSON-8_L5.9-W5.2-P1.27-BL-1"
+		(property "Footprint" "custom_lib:TDSON-8_L5.9-W5.2-P1.27-BL-1"
 			(at 41.91 157.48 0)
 			(hide yes)
