File: pcb/PowerSupply.kicad_pcb (KiCad board)
At the start: 2 copper layers, 8 parts, among them SW1 SW_Push_DPDT, U1 LM5176PWP, U3 CH224K

Commit message: 所有封装
Parts:
- removed D2, D3: ~, Diode_THT:D_DO-41_SOD81_P10.16mm_Horizontal
- added C1: 22u 20V, Capacitor_SMD:CP_Elec_5x5.4, F.Cu at (158.9, 88.4)
- added C2: 22u 20V, Capacitor_SMD:C_Elec_5x5.4, F.Cu at (119.5, 101.8)
- added C26: 100n, Capacitor_SMD:C_0805_2012Metric, F.Cu at (126.5, 86.5)
- added C27: 100n 63V, Capacitor_SMD:C_0805_2012Metric, F.Cu at (126.5, 89.5)
- added C28: 1u, Capacitor_SMD:C_0805_2012Metric, F.Cu at (126.5, 92.5)
- added C29: 100n, Capacitor_SMD:C_0805_2012Metric, F.Cu at (126.5, 95.5)
- added C3: 22u 20V, Capacitor_SMD:CP_Elec_5x5.4, F.Cu at (158.9, 95.2)
- added C30: 100n, Capacitor_SMD:C_0805_2012Metric, F.Cu at (126.5, 98.5)
- added C31: 47p, Capacitor_SMD:C_0805_2012Metric, F.Cu at (126.5, 101.5)
- added C32: 100n, Capacitor_SMD:C_0805_2012Metric, F.Cu at (130.9, 86.5)
- added C34: 10n, Capacitor_SMD:C_0805_2012Metric, F.Cu at (130.9, 89.5)
- added C35: 1u, Capacitor_SMD:C_0805_2012Metric, F.Cu at (130.9, 92.5)
- added C36: 4.7u, Capacitor_SMD:C_0805_2012Metric, F.Cu at (130.9, 95.5)
- added C37: 4.7u, Capacitor_SMD:C_0805_2012Metric, F.Cu at (130.9, 98.5)
- added C38: 4.7u, Capacitor_SMD:C_0805_2012Metric, F.Cu at (130.9, 101.5)
- added C39: 4.7u, Capacitor_SMD:C_0805_2012Metric, F.Cu at (135.4, 86.5)
- added C4: 22u 20V, Capacitor_SMD:CP_Elec_5x5.4, F.Cu at (158.9, 102.1)
- added C40: 4.7u, Capacitor_SMD:C_0805_2012Metric, F.Cu at (135.4, 89.5)
- added C45: 1u, Capacitor_SMD:C_1206_3216Metric, F.Cu at (112.5, 86.4)
- added C46: 1u, Capacitor_SMD:C_1206_3216Metric, F.Cu at (112.5, 89.8)
- added C47: 1u, Capacitor_SMD:C_1206_3216Metric, F.Cu at (112.5, 93.1)
- added C48: 1u, Capacitor_SMD:C_1206_3216Metric, F.Cu at (112.5, 96.5)
- added C49: 1u, Capacitor_SMD:C_1206_3216Metric, F.Cu at (112.5, 99.8)
- added C5: 100u 50V, Capacitor_SMD:CP_Elec_10x10.5, F.Cu at (117.1, 54.6)
- added C53: 240p, Capacitor_SMD:C_0805_2012Metric, F.Cu at (135.4, 92.5)
- added C54: 33n, Capacitor_SMD:C_0805_2012Metric, F.Cu at (135.4, 95.5)
- added C55: 560p, Capacitor_SMD:C_0805_2012Metric, F.Cu at (135.4, 98.5)
- added C6: 100u 50V, Capacitor_SMD:CP_Elec_10x10.5, F.Cu at (117.1, 66.7)
- added C7: 100u 50V, Capacitor_SMD:CP_Elec_10x10.5, F.Cu at (117.1, 78.7)
- added D6: SS310, Diode_SMD:D_SMA, F.Cu at (119.4, 96.1)
- added D7: LED, LED_SMD:LED_0805_2012Metric, F.Cu at (156.3, 74.0)
- added L2: 4.7u, Inductor_SMD:L_TaiTech_TMPC1265_13.5x12.5mm, F.Cu at (153.6, 55.6)
- added Q5: Q_NMOS, lcsc_pro:TDSON-8_L5.9-W5.2-P1.27-BL-1, F.Cu at (127.7, 81.9)
- added Q6: Q_NMOS, lcsc_pro:TDSON-8_L5.9-W5.2-P1.27-BL-1, F.Cu at (134.3, 81.9)
- added Q7: Q_NMOS, lcsc_pro:TDSON-8_L5.9-W5.2-P1.27-BL-1, F.Cu at (140.9, 81.9)
- added Q8: Q_NMOS, lcsc_pro:TDSON-8_L5.9-W5.2-P1.27-BL-1, F.Cu at (147.5, 81.9)
- added R16: 470k, Resistor_SMD:R_1206_3216Metric, F.Cu at (140.4, 86.6)
- added R17: 130k, Resistor_SMD:R_1206_3216Metric, F.Cu at (140.4, 89.9)
- added R18: 10R, Resistor_SMD:R_1206_3216Metric, F.Cu at (140.4, 93.2)
- added R19: 2k, Resistor_SMD:R_1206_3216Metric, F.Cu at (140.4, 96.6)
- added R21: 93.1k, Resistor_SMD:R_1206_3216Metric, F.Cu at (146.0, 86.6)
- added R22: 8m, Resistor_SMD:R_2512_6332Metric, F.Cu at (158.5, 65.1)
- added R23: 100, Resistor_SMD:R_1206_3216Metric, F.Cu at (146.0, 89.9)
- added R24: 100, Resistor_SMD:R_1206_3216Metric, F.Cu at (146.0, 93.2)
- added R25: 1.5k, Resistor_SMD:R_1206_3216Metric, F.Cu at (146.0, 96.6)
- added R26: 5.1k, Resistor_SMD:R_1206_3216Metric, F.Cu at (151.6, 86.6)
- added R27: 100, Resistor_SMD:R_1206_3216Metric, F.Cu at (151.6, 89.9)
- added R28: 100, Resistor_SMD:R_1206_3216Metric, F.Cu at (151.6, 93.2)
- added R29: 8m, Resistor_SMD:R_2512_6332Metric, F.Cu at (158.5, 70.0)
- added R30: 10k, Resistor_SMD:R_1206_3216Metric, F.Cu at (151.6, 96.6)
- added RV1: 100k, lcsc_pro:RES-ADJ-TH_RK097111080R, F.Cu at (129.6, 51.2)
- added RV2: 100k, lcsc_pro:RES-ADJ-TH_RK097111080R, F.Cu at (140.4, 51.2)
- moved R20 81.5 mm to (176.9, 56.7)
- moved U3 81.4 mm to (170.0, 51.8)
- moved U1 80.4 mm to (149.9, 68.3)
- moved SW1 62.6 mm to (170.5, 59.5)
- moved D4 49.6 mm to (119.4, 87.0)
- moved D5 49.6 mm to (119.4, 91.6)
Connections:
- U1 pad 11: fb -> /FB
- U1 pad 12: Vout -> LM5176_VOUT
- U1 pad 13: isns- -> /ISNS-
- U1 pad 14: isns+ -> /ISNS+
- U1 pad 15: csg -> /CSG
- U1 pad 16: cs -> /CS
- U1 pad 17: pgood -> /PGOOD
- U1 pad 18: q4-2 -> /SW2
- U1 pad 19: hdrv2 -> /HDRV2
- U1 pad 21: ldrv2 -> /LDRV2
- U1 pad 24: bias -> /BIAS
- U1 pad 25: ldrv1 -> /LDRV1
- U1 pad 27: hdrv1 -> /HDRV1
- U1 pad 29: powerPAD -> GND
- U1 pad 4: mode -> /MODE
- U1 pad 5: GND -> /DITH
- U1 pad 6: rt/sync -> /RT_SYNC
- U1 pad 7: slope -> /SLOPE
- U1 pad 9: comp -> /COMP

Commit message: 调整元件参数
Parts:
- removed C30, C32: 100n, Capacitor_SMD:C_0805_2012Metric
- removed C31: 47p, Capacitor_SMD:C_0805_2012Metric
- removed C34: 10n, Capacitor_SMD:C_0805_2012Metric
- removed C35: 1u, Capacitor_SMD:C_0805_2012Metric
- removed C36, C37, C38, C39, C40: 4.7u, Capacitor_SMD:C_0805_2012Metric
- removed C45, C46, C47, C48, C49: 1u, Capacitor_SMD:C_1206_3216Metric
- removed C53: 240p, Capacitor_SMD:C_0805_2012Metric
- removed C54: 33n, Capacitor_SMD:C_0805_2012Metric
- removed C55: 560p, Capacitor_SMD:C_0805_2012Metric
- removed D5, D6: SS310, Diode_SMD:D_SMA
- removed D7: LED, LED_SMD:LED_0805_2012Metric
- removed L2: 4.7u, Inductor_SMD:L_TaiTech_TMPC1265_13.5x12.5mm
- removed Q5, Q6, Q7, Q8: Q_NMOS, lcsc_pro:TDSON-8_L5.9-W5.2-P1.27-BL-1
- removed R16: 470k, Resistor_SMD:R_1206_3216Metric
- removed R17: 130k, Resistor_SMD:R_1206_3216Metric
- removed R18: 10R, Resistor_SMD:R_1206_3216Metric
- removed R19: 2k, Resistor_SMD:R_1206_3216Metric
- removed R20: 10k, Capacitor_SMD:C_1206_3216Metric
- removed R21: 93.1k, Resistor_SMD:R_1206_3216Metric
- removed R22, R29: 8m, Resistor_SMD:R_2512_6332Metric
- removed R23, R24, R27, R28: 100, Resistor_SMD:R_1206_3216Metric
- removed R25: 1.5k, Resistor_SMD:R_1206_3216Metric
- removed R26: 5.1k, Resistor_SMD:R_1206_3216Metric
- removed R30: 10k, Resistor_SMD:R_1206_3216Metric
- removed U3: CH224K, Package_SO:SSOP-10-1EP_3.9x4.9mm_P1mm_EP2.1x3.3mm
- added C10: 2.2u 100V, Capacitor_SMD:C_1206_3216Metric, F.Cu at (120.9, 86.3)
- added C11: 2.2u 100V, Capacitor_SMD:C_1206_3216Metric, F.Cu at (120.9, 89.6)
- added C12: 33n, Capacitor_SMD:C_0805_2012Metric, F.Cu at (146.2, 109.8)
- added C13: 100n, Capacitor_SMD:C_0805_2012Metric, F.Cu at (150.6, 100.8)
- added C14: 10n, Capacitor_SMD:C_0805_2012Metric, F.Cu at (150.6, 103.8)
- added C15: 2.2u 100V, Capacitor_SMD:C_1206_3216Metric, F.Cu at (120.9, 93.0)
- added C16: 2.2u 100V, Capacitor_SMD:C_1206_3216Metric, F.Cu at (120.9, 96.3)
- added C17: 330p, Capacitor_SMD:C_0805_2012Metric, F.Cu at (150.6, 106.8)
- added C18: 2.2u 100V, Capacitor_SMD:C_1206_3216Metric, F.Cu at (120.9, 99.7)
- added C19: 2.2u 100V, Capacitor_SMD:C_1206_3216Metric, F.Cu at (120.9, 103.0)
- added C20: 2.2u 100V, Capacitor_SMD:C_1206_3216Metric, F.Cu at (120.9, 106.4)
- added C21: 2.2u 100V, Capacitor_SMD:C_1206_3216Metric, F.Cu at (120.9, 109.7)
- added C22: 470p, Capacitor_SMD:C_0805_2012Metric, F.Cu at (150.6, 109.8)
- added C23: 100u 63V, Capacitor_SMD:CP_Elec_8x10.5, F.Cu at (111.4, 54.7)
- added C24: 100u 63V, Capacitor_SMD:CP_Elec_8x10.5, F.Cu at (111.4, 64.7)
- added C25: 100u 63V, Capacitor_SMD:CP_Elec_8x10.5, F.Cu at (111.4, 74.8)
- added C8: 2.2u 100V, Capacitor_SMD:C_1206_3216Metric, F.Cu at (120.9, 79.6)
- added C9: 2.2u 100V, Capacitor_SMD:C_1206_3216Metric, F.Cu at (120.9, 82.9)
- added D1: SS14, Diode_SMD:D_SMA, F.Cu at (143.7, 51.9)
- added D2: SS310, Diode_SMD:D_SMA, F.Cu at (143.7, 56.5)
- added D3: SS310, Diode_SMD:D_SMA, F.Cu at (143.7, 61.0)
- added L1: 4.7u, Inductor_SMD:L_TaiTech_TMPC1265_13.5x12.5mm, F.Cu at (131.6, 106.3)
- added Q1: Q_NMOS, lcsc_pro:TDSON-8_L5.9-W5.2-P1.27-BL-1, F.Cu at (127.2, 82.9)
- added Q2: Q_NMOS, lcsc_pro:TDSON-8_L5.9-W5.2-P1.27-BL-1, F.Cu at (133.8, 82.9)
- added Q3: Q_NMOS, lcsc_pro:TDSON-8_L5.9-W5.2-P1.27-BL-1, F.Cu at (140.4, 82.9)
- added Q4: Q_NMOS, lcsc_pro:TDSON-8_L5.9-W5.2-P1.27-BL-1, F.Cu at (147.0, 82.9)
- added R1: 100, Resistor_SMD:R_1206_3216Metric, F.Cu at (126.6, 87.7)
- added R10: 2k, Resistor_SMD:R_1206_3216Metric, F.Cu at (132.2, 97.6)
- added R11: 100, Resistor_SMD:R_1206_3216Metric, F.Cu at (137.8, 87.7)
- added R12: 20k, Resistor_SMD:R_1206_3216Metric, F.Cu at (137.8, 91.0)
- added R13: 1.5k, Resistor_SMD:R_1206_3216Metric, F.Cu at (137.8, 94.3)
- added R14: 5.1k, Resistor_SMD:R_1206_3216Metric, F.Cu at (137.8, 97.6)
- added R15: 10k, Capacitor_SMD:C_1206_3216Metric, F.Cu at (166.4, 57.8)
- added R2: 100, Resistor_SMD:R_1206_3216Metric, F.Cu at (126.6, 91.0)
- added R3: 249k, Resistor_SMD:R_1206_3216Metric, F.Cu at (126.6, 94.3)
- added R4: 75k, Resistor_SMD:R_1206_3216Metric, F.Cu at (126.6, 97.6)
- added R5: 10R, Resistor_SMD:R_1206_3216Metric, F.Cu at (132.2, 87.7)
- added R6: 8m, Resistor_SMD:R_2512_6332Metric, F.Cu at (144.9, 88.5)
- added R7: 93.1k, Resistor_SMD:R_1206_3216Metric, F.Cu at (132.2, 91.0)
- added R8: 100, Resistor_SMD:R_1206_3216Metric, F.Cu at (132.2, 94.3)
- added R9: 8m, Resistor_SMD:R_2512_6332Metric, F.Cu at (144.9, 93.4)
- added U2: CH224K, Package_SO:SSOP-10-1EP_3.9x4.9mm_P1mm_EP2.1x3.3mm, F.Cu at (159.5, 52.9)
- C1: value 22u 20V -> 47p; footprint Capacitor_SMD:CP_Elec_5x5.4 -> Capacitor_SMD:C_0805_2012Metric
- C2: value 22u 20V -> 1u; footprint Capacitor_SMD:C_Elec_5x5.4 -> Capacitor_SMD:C_0805_2012Metric
- C26, C29: value 100n -> 100u 63V; footprint Capacitor_SMD:C_0805_2012Metric -> Capacitor_SMD:CP_Elec_8x10.5
- C27: value 100n 63V -> 100u 63V; footprint Capacitor_SMD:C_0805_2012Metric -> Capacitor_SMD:CP_Elec_8x10.5
- C28: value 1u -> 100u 63V; footprint Capacitor_SMD:C_0805_2012Metric -> Capacitor_SMD:CP_Elec_8x10.5
- C3: value 22u 20V -> 100n 63V; footprint Capacitor_SMD:CP_Elec_5x5.4 -> Capacitor_SMD:C_0805_2012Metric
- C4: value 22u 20V -> 330n; footprint Capacitor_SMD:CP_Elec_5x5.4 -> Capacitor_SMD:C_0805_2012Metric
- C5, C6: value 100u 50V -> 100n; footprint Capacitor_SMD:CP_Elec_10x10.5 -> Capacitor_SMD:C_0805_2012Metric
- C7: value 100u 50V -> 1u; footprint Capacitor_SMD:CP_Elec_10x10.5 -> Capacitor_SMD:C_0805_2012Metric
- D4: value SS14 -> LED; footprint Diode_SMD:D_SMA -> LED_SMD:LED_0805_2012Metric
- moved C5 54.5 mm to (146.2, 100.8)
- moved C6 47.1 mm to (146.2, 103.8)
- moved C7 40.4 mm to (146.2, 106.8)
- moved D4 25.6 mm to (142.8, 97.4)
- moved C29 24.6 mm to (111.4, 115.0)
- moved C2 22.3 mm to (141.7, 103.8)
- moved C1 21.2 mm to (141.7, 100.8)
- moved C3 20.7 mm to (141.7, 106.8)
- moved C28 19.5 mm to (111.4, 104.9)
- moved C4 18.8 mm to (141.7, 109.8)
- moved C27 16.0 mm to (111.4, 94.9)
- moved C26 15.1 mm to (111.4, 84.8)
- moved SW1 10.6 mm to (160.0, 60.5)
- moved RV1 6.24 mm to (123.5, 52.3)
- moved RV2 6.24 mm to (134.2, 52.3)
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Connections:
- C1 pad 1: USB_VBUS -> /CSG
- C1 pad 2: GNDPWR -> /CS
- C2 pad 1: USB_VBUS -> GND
- C2 pad 2: GNDPWR -> /VCC
- C26 pad 1: GND -> LM5176_VOUT
- C26 pad 2: /SS -> GNDPWR
- C27 pad 1: GND -> LM5176_VOUT
- C27 pad 2: /VIN -> GNDPWR
- C28 pad 1: GND -> LM5176_VOUT
- C28 pad 2: /VCC -> GNDPWR
- C29 pad 1: /SW1 -> LM5176_VOUT
- C29 pad 2: /BOOT1 -> GNDPWR
- C3 pad 1: USB_VBUS -> GND
- C3 pad 2: GNDPWR -> /VIN
- C4 pad 1: USB_VBUS -> GND
- C4 pad 2: GNDPWR -> /SS
- C5 pad 1: unconnected-(C5-Pad1) -> /SW1
- C5 pad 2: unconnected-(C5-Pad2) -> /BOOT1
- C6 pad 1: LM5176_VOUT -> /SW2
- C6 pad 2: GNDPWR -> /BOOT2
- C7 pad 1: LM5176_VOUT -> /ISNS+
- C7 pad 2: GNDPWR -> /ISNS-
- D4 pad 1: Net-(D4-K) -> GND
- D4 pad 2: USB_VBUS -> /PGOOD
- RV1 pad 1: LM5176_VOUT -> /RT_SYNC
- RV1 pad 2: LM5176_VOUT -> /RT_SYNC
- RV1 pad 3: /FB -> GND
- RV2 pad 1: /RT_SYNC -> LM5176_VOUT
- RV2 pad 2: /RT_SYNC -> LM5176_VOUT
- RV2 pad 3: GND -> /FB
