File: pcb/PowerSupply.kicad_pcb (KiCad board)
At the start: 2 copper layers, 66 parts, among them J1 USB_C_Receptacle_PowerOnly_6P, Q1 Q_NMOS, Q2 Q_NMOS, Q3 Q_NMOS, Q4 Q_NMOS, SW1 SW_DIP_x03, U1 LM5176PWP, U2 CH224K

Commit message: 添加6p typec沉板
Parts:
- J1: footprint Connector_USB:USB_C_Receptacle_GCT_USB4125-xx-x-0190_6P_TopMnt_Horizontal -> lcsc_pro:USB-TYPE-C-SMD_TYPE-C
Other:
- board outline added: 6.6 x 9.2 mm

Commit message: 叫信息
Parts:
- removed SW1: SW_DIP_x03, Button_Switch_SMD:SW_DIP_SPSTx03_Slide_6.7x9.18mm_W8.61mm_P2.54mm_LowProfile
- added SW2: SW_DIP_x03, Button_Switch_SMD:SW_DIP_SPSTx03_Slide_6.7x9.18mm_W8.61mm_P2.54mm_LowProfile, F.Cu at (237.3, 103.5)
- moved D5 56.3 mm to (245.9, 99.5)
- moved C30 51.4 mm to (245.8, 102.5)
- moved R18 28.2 mm to (233.2, 119.2)
- moved R16 28.2 mm to (233.2, 113.3)
- moved R19 28.2 mm to (233.2, 122.1)
- moved R15 28.2 mm to (233.2, 110.3)
- moved R17 28.2 mm to (233.2, 116.2)
- moved R20 28.2 mm to (233.2, 125.1)
- moved U2 22.3 mm to (240.0, 121.0)
- moved J1 3.90 mm to (242.0, 112.2), turned to 0 degrees
Other:
- board size 6.6 x 9.2 mm -> 9.2 x 6.6 mm

Commit message: pcb初版
Parts:
- moved J1 21.6 mm to (220.5, 114.0), turned to -90 degrees
- moved SW2 18.8 mm to (252.8, 114.0)
- moved C30 12.3 mm to (236.1, 110.0)
- moved R18 11.6 mm to (243.6, 114.0)
- moved R17 11.2 mm to (243.6, 112.0)
- moved D5 10.5 mm to (241.5, 109.1), turned to 90 degrees
- moved R20 10.3 mm to (231.1, 115.0), turned to 180 degrees
- moved R19 9.39 mm to (231.1, 113.0), turned to 180 degrees
- moved U2 7.64 mm to (237.0, 114.0)
- moved R16 6.80 mm to (226.4, 113.0)
- moved R15 4.12 mm to (229.1, 110.5)
Routing:
- net VDD: track 0.00 -> 36.7 mm
- net Net-(J1-CC1): track 0.00 -> 26.8 mm
- net Net-(J1-CC2): track 0.00 -> 22.8 mm, vias 0 -> 2
- net Net-(U2-CFG3): track 0.00 -> 19.9 mm, vias 0 -> 1
- net USB_VBUS: track 0.00 -> 18.2 mm, vias 0 -> 1
- net Net-(U2-CFG2): track 0.00 -> 16.3 mm, vias 0 -> 1
- net Net-(U2-CFG1): track 0.00 -> 14.2 mm, vias 0 -> 1
- net Net-(U2-VBUS): track 0.00 -> 12.6 mm, vias 0 -> 1
- net Net-(J1-VBUS-PadA9): track 0.00 -> 11.5 mm, vias 0 -> 1
- net GND: track 0.00 -> 6.97 mm
- net Net-(D5-A): track 0.00 -> 5.85 mm, vias 0 -> 1
- net Net-(D5-K): track 0.00 -> 3.36 mm
Other:
- board size 9.2 x 6.6 mm -> 6.6 x 9.2 mm

Commit message: 总开关电路
Parts:
- added D6: D_Zener, Diode_SMD:D_SOD-123, F.Cu at (92.9, 77.9)
- added Q5: PMOS, lcsc_pro:DFN-8_L5.8-W4.9-P1.27-LS6.1-BL-2, F.Cu at (93.4, 71.8)
- added R24: 5.1k, Resistor_SMD:R_1206_3216Metric, F.Cu at (76.8, 99.2)
- added R25: 5.1k, Resistor_SMD:R_1206_3216Metric, F.Cu at (76.8, 102.5)
- added SW1: SW_Push_DPDT, lcsc_pro:SW-SMD_6P-L9.1-W3.5-P2.50, F.Cu at (95.1, 63.5)
- L1: value 4.7u -> 3.3u
- moved D1 73.1 mm to (83.7, 107.2)
- moved D2 73.1 mm to (83.7, 111.8)
- moved D3 73.1 mm to (83.7, 116.3)
- moved U1 57.6 mm to (91.9, 110.6)
- moved C12 47.5 mm to (69.5, 118.0)
- moved C13 47.5 mm to (73.9, 109.0)
- moved C22 47.5 mm to (73.9, 118.0)
- moved C5 47.5 mm to (69.5, 109.0)
- moved C14 47.5 mm to (73.9, 112.0)
- moved C17 47.5 mm to (73.9, 115.0)
- moved C6 47.5 mm to (69.5, 112.0)
- moved C7 47.5 mm to (69.5, 115.0)
- moved C1 47.5 mm to (65.0, 109.0)
- moved C4 47.5 mm to (65.0, 118.0)
- moved C2 47.5 mm to (65.0, 112.0)
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Connections:
- C11 pad 2: USB_VBUS -> /INPUT
- C16 pad 2: USB_VBUS -> /INPUT
- C19 pad 2: USB_VBUS -> /INPUT
- C21 pad 2: USB_VBUS -> /INPUT
- C24 pad 1: USB_VBUS -> /INPUT
- C9 pad 2: USB_VBUS -> /INPUT
- D1 pad 2: USB_VBUS -> /INPUT
- Q1 pad D: USB_VBUS -> /INPUT
- R10 pad 2: USB_VBUS -> /INPUT
- R3 pad 2: USB_VBUS -> /INPUT

Commit message: 整理封装
Parts:
- removed Q5: PMOS, lcsc_pro:DFN-8_L5.8-W4.9-P1.27-LS6.1-BL-2
- added Q6: Q_PMOS, custom_lib:DFN-8_L5.8-W4.9-P1.27-LS6.1-BL-2, F.Cu at (82.7, 60.0)
- Q1, Q2, Q3, Q4: footprint lcsc_pro:TDSON-8_L5.9-W5.2-P1.27-BL-1 -> custom_lib:TDSON-8_L5.9-W5.2-P1.27-BL-1
- RV1, RV2: footprint lcsc_pro:RES-ADJ-TH_RK097111080R -> custom_lib:RES-ADJ-TH_RK097111080R
- SW1: footprint lcsc_pro:SW-SMD_6P-L9.1-W3.5-P2.50 -> custom_lib:SW-SMD_6P-L9.1-W3.5-P2.50
- moved C4 15.9 mm to (54.4, 106.2)
- moved R11 15.9 mm to (60.6, 90.7)
- moved R12 15.9 mm to (60.6, 94.0)
- moved R25 15.9 mm to (66.2, 90.7)
- moved R4 15.9 mm to (55.0, 90.7)
- moved R5 15.9 mm to (55.0, 94.0)
- moved R6 15.9 mm to (83.7, 40.0)
- moved RV1 15.9 mm to (63.2, 40.1)
- moved RV2 15.9 mm to (73.9, 40.1)
- moved SW1 15.9 mm to (84.4, 51.7)
- moved C20 15.9 mm to (55.0, 66.0)
- moved C22 15.9 mm to (63.3, 106.2)
- moved C27 15.9 mm to (45.5, 82.7)
- moved C18 15.9 mm to (55.0, 59.3)
- moved C23 15.9 mm to (45.5, 42.5)
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
Commit message: ch224k
Parts:
- removed J1: USB_C_Receptacle_PowerOnly_6P, lcsc_pro:USB-TYPE-C-SMD_TYPE-C
- added J2: USB_C_Receptacle_USB2.0_16P, custom_lib:USB-C-SMD_HH-16P-CB-TYPE-C, F.Cu at (157.4, 123.1)
- added REF**: TestPoint_THTPad_D1.0mm_Drill0.5mm, TestPoint:TestPoint_THTPad_D1.0mm_Drill0.5mm, F.Cu at (169.8, 118.0)
- moved SW2 90.9 mm to (164.2, 134.3)
- moved R18 89.6 mm to (155.8, 131.6), turned to 180 degrees
- moved R20 78.3 mm to (155.9, 137.0)
- moved R19 78.2 mm to (155.8, 134.2)
- moved C30 71.9 mm to (164.5, 117.4), turned to 180 degrees
- moved U2 70.9 mm to (166.5, 121.5)
- moved R17 69.9 mm to (174.5, 122.6), turned to 90 degrees
- moved D5 69.7 mm to (172.7, 119.6), turned to 0 degrees
- moved R15 68.1 mm to (161.2, 116.3), turned to 90 degrees
- moved R16 55.3 mm to (172.0, 122.6), turned to 90 degrees
Connections:
- C30 pad 1: VDD -> GND
- C30 pad 2: GND -> Net-(U2-VDD)
- R15 pad 1: Net-(J1-VBUS-PadA9) -> USB_VBUS
- R15 pad 2: VDD -> Net-(U2-VDD)
- SW2 pad 4: VDD -> Net-(U2-VDD)
- SW2 pad 5: VDD -> Net-(U2-VDD)
- SW2 pad 6: VDD -> Net-(U2-VDD)
- U2 pad 1: VDD -> Net-(U2-VDD)
- U2 pad 4: unconnected-(U2-DP-Pad4) -> Net-(U2-DP)
- U2 pad 5: unconnected-(U2-DM-Pad5) -> Net-(U2-DM)
Routing:
- net Net-(U2-VDD): track 0.00 -> 37.5 mm, vias 0 -> 3
- net VDD: track 36.7 -> 0.00 mm
- net Net-(J2-CC1): track 26.8 -> 13.3 mm, vias 0 -> 2
- net Net-(J2-CC2): track 22.8 -> 9.64 mm, vias 2 -> 0
- net Net-(U2-CFG2): track 16.3 -> 28.2 mm, vias 1 -> 2
- net Net-(J1-VBUS-PadA9): track 11.5 -> 0.00 mm, vias 1 -> 0
- net Net-(U2-VBUS): track 12.6 -> 3.56 mm, vias 1 -> 0
- net Net-(U2-DP): track 0.00 -> 8.78 mm, vias 0 -> 2
- net Net-(U2-CFG1): track 14.2 -> 22.1 mm, vias 1 -> 2
- net GND: track 6.97 -> 14.7 mm, vias 0 -> 10
- net Net-(U2-DM): track 0.00 -> 7.16 mm, vias 0 -> 2
- net Net-(D5-A): track 5.85 -> 2.44 mm, vias 1 -> 0
- net Net-(U2-CFG3): track 19.9 -> 22.6 mm, vias 1 -> 2
- net Net-(D5-K): track 3.36 -> 2.59 mm
- net USB_VBUS: track 18.2 -> 18.4 mm, vias 1 -> 8
- added copper zone on F.Cu, net GND
- added copper zone on F.Cu, net USB_VBUS
Other:
- board size 6.6 x 9.2 mm -> 56.9 x 41.2 mm
- copper layers 2 -> 4

Commit message: 还是ch224k
Parts:
- moved C1 158.3 mm to (212.6, 103.8)
- moved C10 158.3 mm to (213.2, 52.5)
- moved C11 158.3 mm to (213.2, 55.8)
- moved C15 158.3 mm to (213.2, 59.2)
- moved C16 158.3 mm to (213.2, 62.5)
- moved C18 158.3 mm to (213.2, 65.9)
- moved C19 158.3 mm to (213.2, 69.2)
- moved C2 158.3 mm to (212.6, 106.8)
- moved C20 158.3 mm to (213.2, 72.6)
- moved C21 158.3 mm to (213.2, 75.9)
- moved C23 158.3 mm to (203.7, 49.1)
- moved C24 158.3 mm to (203.7, 59.2)
- moved C25 158.3 mm to (203.7, 69.2)
- moved C26 158.3 mm to (203.7, 79.3)
- moved C27 158.3 mm to (203.7, 89.3)
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Routing:
- added copper zone on In2.Cu, net USB_VBUS

Commit message: 再修ch224k
Routing:
- net USB_VBUS: track 18.4 -> 23.9 mm
Changed lines of the file:
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@@
 		(capping no)
 		(filling no)
+		(zone_defaults)
 		(pcbplotparams
 			(layerselection 0x00000000_00000000_55555555_5755f5ff)
@@
 		(layer "F.Cu")
 		(net "USB_VBUS")
+	)
+	(segment
+		(start 152 59.95)
+		(end 157.525 59.95)
+		(width 1.1684)
+		(layer "F.Cu")
+		(net "USB_VBUS")
