File: pcb/PowerSupply.kicad_pcb (KiCad board)
At the start: 4 copper layers, 56.9 x 41.2 mm, 72 parts, among them J2 USB_C_Receptacle_USB2.0_16P, Q1 Q_NMOS, Q2 Q_NMOS, Q3 Q_NMOS, Q4 Q_NMOS, Q6 Q_PMOS, SW1 SW_Push_DPDT, SW2 SW_DIP_x03, U1 LM5176PWP, U2 CH224K

Commit message: 更新PCB布局
Parts:
- moved C1 109.3 mm to (106.4, 77.6)
- moved C2 109.3 mm to (106.4, 80.7)
- moved C3 109.3 mm to (106.4, 83.7)
- moved R10 109.3 mm to (112.6, 67.9)
- moved R12 109.3 mm to (112.6, 74.5)
- moved R7 109.3 mm to (112.6, 61.2)
- moved C10 109.3 mm to (107.0, 26.4)
- moved C11 109.3 mm to (107.0, 29.7)
- moved C12 109.3 mm to (110.9, 86.7)
- moved C15 109.3 mm to (107.0, 33.0)
- moved C16 109.3 mm to (107.0, 36.4)
- moved C18 109.3 mm to (107.0, 39.8)
- moved C19 109.3 mm to (107.0, 43.1)
- moved C20 109.3 mm to (107.0, 46.5)
- moved C21 109.3 mm to (107.0, 49.8)
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Routing:
- net /SW1: track 0.00 -> 51.3 mm, vias 0 -> 2
- net Net-(Q3-PadD): track 0.00 -> 40.0 mm
- net /SW2: track 0.00 -> 36.5 mm, vias 0 -> 2
- net /LDRV1: track 0.00 -> 22.8 mm
- net /VCC: track 0.00 -> 21.8 mm, vias 0 -> 1
- net Net-(Q2-PadS): track 0.00 -> 21.4 mm
- net /HDRV2: track 0.00 -> 17.6 mm
- net /HDRV1: track 0.00 -> 15.0 mm
- net LM5176_VOUT: track 0.00 -> 13.9 mm
- net /BOOT1: track 0.00 -> 13.2 mm, vias 0 -> 2
- net /BOOT2: track 0.00 -> 12.3 mm, vias 0 -> 2
- net /LDRV2: track 0.00 -> 12.0 mm
- net /SS: track 0.00 -> 9.41 mm, vias 0 -> 2
- net /ISNS+: track 0.00 -> 7.79 mm
- net /ISNS-: track 0.00 -> 7.19 mm

Commit message: 更新PCB布局
Parts:
- moved C24 129.1 mm to (225.3, 51.5)
- moved C19 111.6 mm to (217.9, 55.4), turned to 90 degrees
- moved C16 110.4 mm to (215.8, 55.4), turned to 90 degrees
- moved C9 109.5 mm to (211.7, 55.4), turned to 90 degrees
- moved C21 106.9 mm to (213.7, 55.4), turned to 90 degrees
- moved C11 104.0 mm to (208.1, 54.2), turned to 180 degrees
- moved C2 102.3 mm to (208.1, 69.4), turned to -90 degrees
Routing:
- net /INPUT: track 0.00 -> 39.4 mm, vias 0 -> 2
- net Net-(Q3-PadD): track 40.0 -> 47.1 mm
- net /VCC: track 21.8 -> 24.7 mm
- net /SW1: track 51.3 -> 52.9 mm

Commit message: 更新
Parts:
- moved C8 143.0 mm to (220.0, 107.3), turned to 90 degrees
- moved C10 137.0 mm to (217.6, 107.3), turned to 90 degrees
- moved C15 131.1 mm to (215.1, 107.3), turned to 90 degrees
- moved C18 125.3 mm to (212.6, 107.3), turned to 90 degrees
- moved C20 119.6 mm to (209.9, 107.3), turned to 90 degrees
- moved R7 98.6 mm to (205.5, 94.4)
- moved C14 95.2 mm to (209.1, 96.8)
- moved C23 93.8 mm to (169.1, 83.7)
- moved C22 90.5 mm to (205.2, 96.8)
- moved C29 76.0 mm to (167.2, 113.7)
- moved C25 71.2 mm to (160.4, 76.5), turned to 90 degrees
- moved C27 70.0 mm to (159.1, 96.5), turned to 180 degrees
- moved C28 69.6 mm to (154.2, 113.7), turned to 180 degrees
- moved C26 67.0 mm to (155.2, 87.2), turned to 180 degrees
- moved C11 44.7 mm to (239.2, 86.5)
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Routing:
- net LM5176_VOUT: track 13.9 -> 72.5 mm, vias 0 -> 2
- net Net-(Q3-PadD): track 47.1 -> 11.1 mm
- net /SLOPE: track 0.00 -> 9.91 mm
- net /MODE: track 0.00 -> 9.37 mm
- net /DITH: track 0.00 -> 5.52 mm
- net /ISNS-: track 7.19 -> 9.32 mm
- net /ISNS+: track 7.79 -> 9.55 mm

Commit message: pcb布局调整
Parts:
- moved C16 128.4 mm to (118.5, 90.5)
- moved C24 128.4 mm to (128.0, 86.6)
- moved Q3 128.4 mm to (109.5, 110.1)
- moved Q4 128.4 mm to (104.0, 110.1)
- moved C11 128.4 mm to (110.8, 89.3)
- moved C18 128.4 mm to (84.2, 110.1)
- moved C2 128.4 mm to (110.8, 104.5)
- moved C21 128.4 mm to (116.4, 90.5)
- moved C22 128.4 mm to (76.8, 99.7)
- moved C4 128.4 mm to (76.8, 101.8)
- moved C5 128.4 mm to (101.0, 101.6)
- moved C6 128.4 mm to (101.0, 105.0)
- moved C8 128.4 mm to (91.6, 110.1)
- moved D3 128.4 mm to (105.8, 105.3)
- moved L1 128.4 mm to (118.8, 103.4)
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Routing:
- net /FB: track 0.00 -> 55.0 mm, vias 0 -> 3
- net USB_VBUS: track 23.9 -> 78.4 mm
- net /RT_SYNC: track 0.00 -> 44.2 mm, vias 0 -> 2
- net /INPUT: track 39.4 -> 73.5 mm
- net Net-(Q2-PadS): track 21.4 -> 45.6 mm, vias 0 -> 3
- net /COMP: track 0.00 -> 21.7 mm, vias 0 -> 2
- net /VISNS: track 0.00 -> 20.4 mm
- net /VIN: track 0.00 -> 18.9 mm
- net /EN_UVLO: track 0.00 -> 17.2 mm, vias 0 -> 2
- net /BIAS: track 0.00 -> 15.6 mm, vias 0 -> 2
- net /CS: track 0.00 -> 14.5 mm, vias 0 -> 2
- net /CSG: track 0.00 -> 13.2 mm, vias 0 -> 2
- net /PGOOD: track 0.00 -> 11.8 mm
- net Net-(D6-A): track 0.00 -> 10.2 mm
- net Net-(R24-Pad1): track 0.00 -> 9.36 mm
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Other:
- board size 56.9 x 41.2 mm -> 97 x 97 mm
