File: pcb/ch224k.kicad_sch (KiCad schematic)
At the start: 0 parts

Commit message: first teach
Parts:
- added R20: 10k, Capacitor_SMD:C_1206_3216Metric, symbol Device:R
- added SW1: SW_Push_DPDT, lcsc_pro:SW-SMD_6P-L9.1-W3.5-P2.50, symbol Switch:SW_Push_DPDT
- added U3: CH224K, Package_SO:SSOP-10-1EP_3.9x4.9mm_P1mm_EP2.1x3.3mm, symbol Interface_USB:CH224K

Commit message: 调整元件参数
Parts:
- renumbered R20 to R15, U3 to U2
Changed lines of the file:
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@@
 		(dnp no)
 		(fields_autoplaced yes)
-		(property "Reference" "R20"
+		(property "Reference" "R15"
 			(at 154.94 58.4199 0)
 			(show_name no)
@@
 			(project "PowerSupply"
 				(path "/3ecbe32c-4290-401a-9b8c-a7a0b4ba8879/52948868-4154-4f87-b260-a7c6d385dce1"
-					(reference "R20")
+					(reference "R15")
 					(unit 1)
 				)
@@
 		(dnp no)
 		(fields_autoplaced yes)
-		(property "Reference" "U3"
+		(property "Reference" "U2"
 			(at 129.1433 80.01 0)
 			(show_name no)
@@
 			(project "PowerSupply"
 				(path "/3ecbe32c-4290-401a-9b8c-a7a0b4ba8879/52948868-4154-4f87-b260-a7c6d385dce1"
-					(reference "U3")
+					(reference "U2")
 					(unit 1)
 				)

Commit message: 提交信息
Parts:
- removed SW1: SW_Push_DPDT, lcsc_pro:SW-SMD_6P-L9.1-W3.5-P2.50, symbol Switch:SW_Push_DPDT
- added C30: 1u, Capacitor_SMD:C_0805_2012Metric, symbol Device:C
- added D5: LED, LED_SMD:LED_0805_2012Metric, symbol Device:LED
- added J1: USB_C_Receptacle_PowerOnly_6P, Connector_USB:USB_C_Receptacle_GCT_USB4125-xx-x-0190_6P_TopMnt_Horizontal, symbol Connector:USB_C_Receptacle_PowerOnly_6P
- added R16, R18, R19, R20: 10k, Resistor_SMD:R_0805_2012Metric, symbol Device:R
- added R17: 5.1k, Resistor_SMD:R_0805_2012Metric, symbol Device:R
- added SW1: SW_DIP_x03, Button_Switch_SMD:SW_DIP_SPSTx03_Slide_6.7x9.18mm_W8.61mm_P2.54mm_LowProfile, symbol Switch:SW_DIP_x03
- R15: value 10k -> 1k; footprint Capacitor_SMD:C_1206_3216Metric -> Resistor_SMD:R_0805_2012Metric
Connections:
- net at R15.1: now also J1.A9 (VBUS), J1.B9 (VBUS)
- net VDD: now reaches R15.2
- net VDD: now also U2.1 (VDD), C30.1, SW1.4, SW1.5, SW1.6
- net at U2.10 (PG): now also D5.1 (K)
- net GND: now reaches U2.11 (GND)
- net GND: now also C30.2, J1.A12 (GND), J1.B12 (GND), J1.SH (SHIELD), R18.2, R19.2, R20.2, SW1.1, SW1.2, SW1.3
- net at U2.2 (CFG2): now also R19.1
- net at U2.3 (CFG3): now also R20.1
- net at U2.6 (CC2): now also J1.B5 (CC2)
- net at U2.7 (CC1): now also J1.A5 (CC1)
- net at U2.8 (VBUS): now also R16.2
- net at U2.9 (CFG1): now also R18.1
- new net: D5.2 (A), R17.2
- new net USB_VBUS: R16.1, R17.1

Commit message: 添加6p typec沉板
Parts:
- J1: footprint Connector_USB:USB_C_Receptacle_GCT_USB4125-xx-x-0190_6P_TopMnt_Horizontal -> lcsc_pro:USB-TYPE-C-SMD_TYPE-C
Changed lines of the file:
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@@
 			)
 		)
-		(property "Footprint" "Connector_USB:USB_C_Receptacle_GCT_USB4125-xx-x-0190_6P_TopMnt_Horizontal"
+		(property "Footprint" "lcsc_pro:USB-TYPE-C-SMD_TYPE-C"
 			(at 106.68 100.33 0)
 			(hide yes)

Commit message: 叫信息
Parts:
- removed SW1: SW_DIP_x03, Button_Switch_SMD:SW_DIP_SPSTx03_Slide_6.7x9.18mm_W8.61mm_P2.54mm_LowProfile, symbol Switch:SW_DIP_x03
- added SW2: SW_DIP_x03, Button_Switch_SMD:SW_DIP_SPSTx03_Slide_6.7x9.18mm_W8.61mm_P2.54mm_LowProfile, symbol Switch:SW_DIP_x03
Connections:
- net VDD: now also SW2.4, SW2.5, SW2.6
- net at R18.1, U2.9 (CFG1): now also SW2.1
- net at R19.1, U2.2 (CFG2): now also SW2.2
- net at R20.1, U2.3 (CFG3): now also SW2.3

Commit message: ch224k
Parts:
- removed J1: USB_C_Receptacle_PowerOnly_6P, lcsc_pro:USB-TYPE-C-SMD_TYPE-C, symbol Connector:USB_C_Receptacle_PowerOnly_6P
- added J2: USB_C_Receptacle_USB2.0_16P, custom_lib:USB-C-SMD_HH-16P-CB-TYPE-C, symbol Connector:USB_C_Receptacle_USB2.0_16P
Connections:
- net GND: now also C30.1, J2.A1 (GND), J2.A12 (GND), J2.B1 (GND), J2.B12 (GND), J2.SH (SHIELD); no longer C30.2
- net USB_VBUS: now also R15.1, J2.A4 (VBUS), J2.A9 (VBUS), J2.B4 (VBUS), J2.B9 (VBUS)
- net at U2.7 (CC1): now also J2.A5 (CC1)
- net at U2.6 (CC2): now also J2.B5 (CC2)
- net at U2.4 (DP): now also J2.A6 (D+), J2.B6 (D+)
- net at U2.5 (DM): now also J2.A7 (D-), J2.B7 (D-)
- net VDD: no longer names the net of R15.2, SW2.4, SW2.5, SW2.6, U2.1 (VDD)
- net VDD: now also C30.2; no longer C30.1
Other:
- moved on the sheet: R18, R20
